File: Shield_VCU_Board/Shield_VCU_Board.kicad_sch (KiCad schematic)
At the start: 153 parts, among them J1 Conn_02x10_Odd_Even, J10 TP, J11 Molex_connector_40pin, J12 TFT Wire, J15 Conn_01x04_Socket, J2 Conn_02x10_Odd_Even, J3 Conn_02x09_Odd_Even, J4 Conn_02x09_Odd_Even, J5 Conn_02x09_Odd_Even, J6 Conn_02x10_Odd_Even, J7 Molex: 4pin, J8 Conn_ToSpeaker, U1 AS1115-BSST, U2 SN74LVC1G125DBV, U3 MC74HC14A, U4 TPA6205A1, U5 TLV76133DCY, U6 TLV76150DCY, U7 FT812, U8 TLV76133DCY, U9 TLV76133DCY, Y1 12MHz, Y2 SGM3766YTN5G

Commit message: DSPL update version - Done
+ TestPins added
Parts:
- removed 7U0, 7U1, 7U2, 7U3, 7U4, 7U5, 7U6, 7U7: HDSP-7803, Display_7Segment:HDSP-7801, symbol Display_Character:HDSP-7803
- removed C12: 0.1uF, symbol Device:C
- removed C13: 4.7uF, symbol Device:C_Polarized
- removed C38, C39: 2.2nF, symbol Device:C_Small
- removed J10: TP, symbol Connector:Conn_01x04_Pin
- removed J7: Molex: 4pin, symbol Connector:Conn_01x04_Socket
- added 7U1, 7U2, 7U3, 7U4, 7U5, 7U6, 7U7, 7U8: HDSP-7803_EVR, Display_7Segment:HDSP-7801, symbol A_GHST_Lib:HDSP-7803_EVR
- added C12: 0.1uF, symbol Device:C_Small
- added C13: 4.7uF, symbol Device:C_Polarized_Small
- added J13: Molex_x06_Socket, symbol Connector:Conn_01x06_Socket
- added J9: Wire_x06_Pin, symbol Connector:Conn_01x06_Pin
- added R55, R56: 4.7k, symbol Device:R_Small
- added R57, R58, R59, R60: 33R, symbol Device:R_Small
- added R61, R63: 1k, symbol Device:R_Small
- added R62: 100k, symbol Device:R_Small
- added R64: 47k, symbol Device:R_Small
- added TP1, TP10, TP11, TP12, TP13, TP14, TP15, TP16, TP17, TP2, TP3, TP4, TP5, TP6, TP7, TP8, TP9: TestPoint, symbol Connector:TestPoint
- C36: value 2.2nF -> 0.1uF
- C37: value 2.2nF -> 27pF
- R6: value 1k -> 33R
- RTP1: value Resistive Touch Panel -> 1.0K-FX-06PWB
Connections:
- net 3V3_DSPL is gone; now on net 3V3_7seg: C16.1, C17.1, C18.1, C19.1, C20.1, C34.1, C40.1, C41.1, C7.1, D10.2 (A), J11.4 (Pin_4), R16.1, R20.1, R21.1, R22.1, U3.14 (VCC), U7.11 (VCCIO1), U7.19 (VCC), U7.21 (VCC), U7.22 (VCCIO2), U9.2 (VO)
- net 3V3_SPKR is gone; now on net 3V3_7seg: C28.1, D7.2 (A), FB2.1, R53.1, U5.2 (VO)
- net LED1_GPIO6 is gone; now on net LED1_PTB9: R2.1
- net LED2_GPIO7 is gone; now on net LED2_PTA12: R3.1
- net LED3_GPIO8 is gone; now on net LED3_PTA24: R4.1
- net LED4_GPIO9 is gone; now on net LED4_PTA25: R5.1
- net NXP_IRQ is gone; now on net 7S_NXP_IRQ: J2.20 (Pin_20)
- net NXP_SCL is gone; now on net 7S_NXP_SCL: J2.19 (Pin_19)
- net NXP_SDA is gone; now on net 7S_NXP_SDA: J2.17 (Pin_17)
- net +12V: now also TP8.1
- net 3V3_7seg: now also C36.1, C37.1, J13.1 (Pin_1), R55.1, R56.1, R61.2, R63.2, R64.2, TP2.1, TP3.1, TP4.1
- net 5V_BKLT: now also TP1.1
- net 7S_NXP_IRQ: now also TP7.1
- net 7S_NXP_SCL: now also R56.2, TP5.1
- net 7S_NXP_SDA: now also R55.2, TP6.1
- net Audio_L: now also TP17.1
- net CAN_H_OUT: now also TP9.1
- net CAN_L_OUT: now also TP10.1
- net FT_CS: now also TP13.1
- net FT_INT: now also TP12.1
- net FT_MISO: now also J2.9 (Pin_9), TP15.1; no longer J2.7 (Pin_7)
- net FT_MOSI: now also J2.7 (Pin_7), TP14.1; no longer J2.9 (Pin_9)
- net FT_PD: now also TP11.1
- net FT_T_SCK: now also TP16.1
- net GND: now also C12.2, C13.2, J13.2 (Pin_2), R62.1
- net VOUT1V2: now also C12.1, C13.1
- net at U1.10 (DIG7): now also 7U8.3 (CC), 7U8.8 (CC)
- net at U1.15 (SEGA): now also 7U1.7 (A), 7U2.7 (A), 7U3.7 (A), 7U4.7 (A), 7U5.7 (A), 7U6.7 (A), 7U7.7 (A), 7U8.7 (A)
- net at U1.16 (SEGF): now also 7U1.9 (F), 7U2.9 (F), 7U3.9 (F), 7U4.9 (F), 7U5.9 (F), 7U6.9 (F), 7U7.9 (F), 7U8.9 (F)
- net at U1.17 (SEGB): now also 7U1.6 (B), 7U2.6 (B), 7U3.6 (B), 7U4.6 (B), 7U5.6 (B), 7U6.6 (B), 7U7.6 (B), 7U8.6 (B)
- net at U1.18 (SEGG): now also 7U1.10 (G), 7U2.10 (G), 7U3.10 (G), 7U4.10 (G), 7U5.10 (G), 7U6.10 (G), 7U7.10 (G), 7U8.10 (G)
- net at U1.2 (DIG0): now also 7U1.3 (CC)
- net at U1.20 (SEGC): now also 7U1.4 (C), 7U2.4 (C), 7U3.4 (C), 7U4.4 (C), 7U5.4 (C), 7U6.4 (C), 7U7.4 (C), 7U8.4 (C)
- net at U1.21 (SEGE): now also 7U1.1 (E), 7U2.1 (E), 7U3.1 (E), 7U4.1 (E), 7U5.1 (E), 7U6.1 (E), 7U7.1 (E), 7U8.1 (E)
- net at U1.22 (SEGDP): now also 7U1.5 (DP), 7U2.5 (DP), 7U3.5 (DP), 7U4.5 (DP), 7U5.5 (DP), 7U6.5 (DP), 7U7.5 (DP), 7U8.5 (DP)
- net at U1.23 (SEGD): now also 7U1.2 (D), 7U2.2 (D), 7U3.2 (D), 7U4.2 (D), 7U5.2 (D), 7U6.2 (D), 7U7.2 (D), 7U8.2 (D)
- net at U1.3 (DIG1): now also 7U2.3 (CC), 7U2.8 (CC)
- net at U1.4 (DIG2): now also 7U3.3 (CC), 7U3.8 (CC)
- net at U1.5 (DIG3): now also 7U4.3 (CC), 7U4.8 (CC)
- net at U1.7 (DIG4): now also 7U5.3 (CC), 7U5.8 (CC)
- net at U1.8 (DIG5): now also 7U6.3 (CC), 7U6.8 (CC)
- net at U1.9 (DIG6): now also 7U7.3 (CC), 7U7.8 (CC)
- net at U7.23 (CTP_SCL): now also R57.1; no longer J11.37 (Pin_37)
- net at U7.24 (CTP_SDA): now also R58.1; no longer J11.40 (Pin_40)
- net at RTP1.1 (VDD): now also J9.1 (Pin_1)
- net at RTP1.2 (GND): now also J9.2 (Pin_2)
- net at RTP1.3 (SCL): now also J9.3 (Pin_3)
- net at RTP1.4 (SDA): now also J9.4 (Pin_4)
- net LED1_PTB9: now reaches J2.10 (Pin_10)
- net LED2_PTA12: now reaches J2.4 (Pin_4)
- net LED3_PTA24: now reaches J2.6 (Pin_6)
- net LED4_PTA25: now reaches J2.8 (Pin_8)
- net at LCD1.37 (NC(XR)): no longer J12.37 (Pin_37)
- net at LCD1.38 (NC(YD)): no longer J12.38 (Pin_38)
- net at LCD1.39 (NC(XL)): no longer J12.39 (Pin_39)
- net at LCD1.40 (NC(YU)): no longer J12.40 (Pin_40)
- new net: R60.1, U7.25 (CTP_RST_N)
- new net: R59.1, U7.26 (CTP_INT_N)
- new net: J13.6 (Pin_6), R60.2, R62.2
- new net: J13.3 (Pin_3), R57.2, R61.1
- new net: J9.5 (Pin_5), RTP1.5 (/INT)
- new net: J9.6 (Pin_6), RTP1.6 (/RESET)
- new net: J13.5 (Pin_5), R59.2, R64.1
- new net: J13.4 (Pin_4), R58.2, R63.1
- now unconnected: J11.38 (Pin_38), J11.39 (Pin_39)
- no-connect marks 24 -> 32
Other:
- note added: "Test points: -Iesirile de la regulatoarele de tensiune -Pinii de SCL, SDA si IRQ de la 7seg -Intrarea de 12v -Pinii de PD, INT, SCK, MISO, MOSI, CS, AUDIO_L de la cipul display-ului -Pinii de CAN"
- note removed: "State LED"
- moved on the sheet: C14, C15, C16, C17, C18, C19, C20, C35, C40, C41, C7, J11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

Commit message: Error corrections
Parts:
- removed Buton_Activation_Logic, Power_Supply: Conn_01x02_Socket, symbol Connector:Conn_01x02_Socket
- removed U4: TPA6205A1, Package_DFN_QFN:Texas_S-PVQFN-N16_EP2.7x2.7mm_ThermalVias, symbol New_Library:TPA6205A1
- removed U7: FT812, symbol New_Library:FT812
- added J10: Main_Supply, symbol Connector:Conn_01x02_Socket
- added J7: Button_Activation_Logic, symbol Connector:Conn_01x02_Socket
- added U4: TPA6205A1, symbol A_GHST_Lib:TPA6205A1
- added U7: FT812, symbol A_GHST_Lib:FT812
- renumbered TP2 to AUDV3.3, TP1 to BKLTV5, TP9 to CAN_H1, TP10 to CAN_L1, TP4 to DSPLV3.3, TP7 to IRQ7, TP5 to SCL7, TP6 to SDA7, TP3 to SEGV3.3, TP8 to V12
Connections:
- net MT_SPI_SCK is gone; now on net MC_SPI_SCK: J2.11 (Pin_11)
- net +12V: now also J10.2 (Pin_2)
- net 3V3_7seg: no longer AUDV3.3.1, C16.1, C17.1, C18.1, C19.1, C20.1, C28.1, C34.1, C36.1, C37.1, C40.1, C41.1, C7.1, D10.2 (A), D7.2 (A), DSPLV3.3.1, FB2.1, J11.4 (Pin_4), J13.1 (Pin_1), R16.1, R20.1, R21.1, R22.1, R53.1, R61.2, R63.2, R64.2, U3.14 (VCC), U5.2 (VO), U9.2 (VO)
- net Audio_L: now also U7.3 (AUDIO_L)
- net BL_PWM: now also U7.28 (BACKLIGHT)
- net FT_CS: now also U7.8 (CS_N)
- net FT_INT: now also U7.13 (INT_N)
- net FT_MISO: now also U7.6 (MISO)
- net FT_MOSI: now also U7.7 (MOSI)
- net FT_PD: now also U7.14 (PD_N)
- net FT_T_SCK: now also U7.5 (SCK)
- net GND: now also J10.1 (Pin_1), U7.18 (GND), U7.27 (GND), U7.4 (GND), U7.42 (GND), U7.EP
- net GNDA: now also U4.7 (GND), U4.9 (GND)
- net at 7U8.3 (CC), U1.10 (DIG7): no longer 7U8.8 (CC)
- net at 7U2.3 (CC), U1.3 (DIG1): no longer 7U2.8 (CC)
- net at 7U3.3 (CC), U1.4 (DIG2): no longer 7U3.8 (CC)
- net at 7U4.3 (CC), U1.5 (DIG3): no longer 7U4.8 (CC)
- net at 7U5.3 (CC), U1.7 (DIG4): no longer 7U5.8 (CC)
- net at 7U6.3 (CC), U1.8 (DIG5): no longer 7U6.8 (CC)
- net at 7U7.3 (CC), U1.9 (DIG6): no longer 7U7.8 (CC)
- net at R10.1, R11.1: now also U4.1 (SHDN)
- net at J8.1 (Pin_1), R15.1: now also U4.5 (VO+)
- net at R14.2, R15.2: now also U4.4 (IN-)
- net at C5.2: now also U4.2 (BYPASS)
- net at R12.1, R13.2: now also U4.3 (IN+)
- net at J8.2 (Pin_2), R13.1: now also U4.8 (VO-)
- net at R49.1: now also U7.1 (R1)
- net at C14.1, Y1.1: now also U7.16 (X1/CLK)
- net at C15.1, Y1.3: now also U7.17 (X2)
- net at R50.1: now also U7.2 (R0)
- net at R57.1: now also U7.23 (CTP_SCL)
- net at R58.1: now also U7.24 (CTP_SDA)
- net at R60.1: now also U7.25 (CTP_RST_N)
- net at R59.1: now also U7.26 (CTP_INT_N)
- net at R27.1: now also U7.29 (DE)
- net at R26.1: now also U7.30 (VSYNC)
- net at R25.1: now also U7.31 (HSYNC)
- net at R24.1: now also U7.32 (DISP)
- net at R23.1: now also U7.33 (PCLK)
- net at R28.1: now also U7.34 (B7)
- net at R29.1: now also U7.35 (B6)
- net at R30.1: now also U7.36 (B5)
- net at R31.1: now also U7.37 (B4)
- net at R32.1: now also U7.38 (B3)
- net at R33.1: now also U7.39 (B2)
- net at R34.1: now also U7.40 (B1)
- net at R35.1: now also U7.41 (B0)
- net at R36.1: now also U7.43 (G7)
- net at R37.1: now also U7.44 (G6)
- net at R38.1: now also U7.45 (G5)
- net at R39.1: now also U7.46 (G4)
- net at R40.1: now also U7.47 (G3)
- net at R41.1: now also U7.48 (G2)
- net at R42.1: now also U7.49 (G1)
- net at R51.1: now also U7.50 (G0)
- net at R43.1: now also U7.51 (R7)
- net at R44.1: now also U7.52 (R6)
- net at R45.1: now also U7.53 (R5)
- net at R46.1: now also U7.54 (R4)
- net at R47.1: now also U7.55 (R3)
- net at R48.1: now also U7.56 (R2)
- net at J2.12 (Pin_12): now also J7.2 (Pin_2)
- net at J2.18 (Pin_18): now also J7.1 (Pin_1)
- net at J12.19 (Pin_19): now also LCD1.19 (G6); no longer LCD1.18 (G6)
- net +3V3_AUD renamed 3V3_SPKR
- net 3V3_SPKR: now also R53.1, U4.6 (VDD)
- net VOUT1V2 renamed +1V2
- net +1V2: now also U7.20 (VOUT1V2)
- new net 3V3_AUD: AUDV3.3.1, C28.1, D7.2 (A), FB2.1, U5.2 (VO)
- new net 3V3_DSPL: C16.1, C17.1, C18.1, C19.1, C20.1, C34.1, C36.1, C37.1, C40.1, C41.1, C7.1, D10.2 (A), DSPLV3.3.1, J11.4 (Pin_4), J13.1 (Pin_1), R16.1, R20.1, R21.1, R22.1, R61.2, R63.2, R64.2, U3.14 (VCC), U7.11 (VCCIO1), U7.19 (VCC), U7.21 (VCC), U7.22 (VCCIO2), U9.2 (VO)
- no-connect marks 32 -> 139
Other:
- note removed: "Test points: -Iesirile de la regulatoarele de tensiune -Pinii de SCL, SDA si IRQ de la 7seg -Intrarea de 12v -Pinii de PD, INT, SCK, MISO, MOSI, CS, AUDIO_L de la cipul display-ului -Pinii de CAN"
- moved on the sheet: AUDV3.3, BKLTV5, DSPLV3.3, H1, H2, H3, H4, SEGV3.3

Commit message: Reverse voltage protection added
Additional:
+4 mounting holes
+corrected 1x resistor value
+AUD pin connected by J2
Parts:
- added D15: 1N5242, Diode_THT:D_DO-201_P15.24mm_Horizontal, symbol Diode:1N53xxB
- added F1: Fuse, symbol Device:Fuse_Small
- added H5: MountingHole_VCU, symbol Mechanical:MountingHole_Pad
- added H6, H7, H8: MountingHole_Pad, symbol Mechanical:MountingHole_Pad
- H3: value MountingHole_Pads -> MountingHole_Car
- R64: value 47k -> 4k7
Connections:
- net +12V: now also D15.1 (K), F1.2; no longer J10.2 (Pin_2)
- net GND: now also D15.2 (A), H5.1, H6.1, H7.1, H8.1
- net NXP_GPIO5: now also J2.2 (Pin_2)
- new net: F1.1, J10.2 (Pin_2)
- no-connect marks 139 -> 138
Other:
- note removed: "Audio shutdown"
- moved on the sheet: J10, V12

Commit message: Protection update
Connections:
- net +12V: no longer F1.2
- net GND: no longer D15.2 (A)
- new net: D15.2 (A), F1.2
Other:
- moved on the sheet: D15, F1, J10
Changed lines of the file:
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@@
 	)
 	(junction
-		(at 193.04 33.02)
-		(diameter 0)
-		(color 0 0 0 0)
-	)
-	(junction
 		(at 27.94 398.78)
 		(diameter 0)
@@
 	)
 	(junction
+		(at 200.66 25.4)
+		(diameter 0)
+		(color 0 0 0 0)
+	)
+	(junction
 		(at 312.42 381)
 		(diameter 0)
@@
 	)
 	(junction
-		(at 200.66 25.4)
-		(diameter 0)
-		(color 0 0 0 0)
-	)
-	(junction
 		(at 302.26 182.88)
 		(diameter 0)
@@
 	)
 	(junction
-		(at 193.04 25.4)
-		(diameter 0)
-		(color 0 0 0 0)
-	)
-	(junction
 		(at 307.34 193.04)
 		(diameter 0)
@@
 	(wire
 		(pts
-			(xy 179.07 33.02) (xy 193.04 33.02)
-		)
-		(stroke
-			(width 0)
-			(type default)
-		)
-	)
-	(wire
-		(pts
 			(xy 334.01 168.91) (xy 334.01 271.78)
 		)
@@
 	(wire
 		(pts
-			(xy 200.66 33.02) (xy 200.66 38.1)
+			(xy 200.66 27.94) (xy 200.66 34.29)
 		)
 		(stroke
@@
 	(wire
 		(pts
+			(xy 195.58 25.4) (xy 200.66 25.4)
+		)
+		(stroke
+			(width 0)
+			(type default)
+		)
+	)
+	(wire
+		(pts
 			(xy 118.11 262.89) (xy 123.19 262.89)
 		)
@@
 	(wire
 		(pts
+			(xy 184.15 25.4) (xy 187.96 25.4)
+		)
+		(stroke
+			(width 0)
+			(type default)
+		)
+	)
+	(wire
+		(pts
 			(xy 533.4 269.24) (xy 541.02 269.24)
 		)
@@
 	(wire
 		(pts
-			(xy 179.07 25.4) (xy 182.88 25.4)
+			(xy 166.37 25.4) (xy 179.07 25.4)
 		)
 		(stroke
@@
 	(wire
 		(pts
-			(xy 179.07 33.02) (xy 179.07 27.94)
-		)
-		(stroke
-			(width 0)
-			(type default)
-		)
-	)
-	(wire
-		(pts
 			(xy 25.4 308.61) (xy 35.56 308.61)
 		)
@@
 	(wire
 		(pts
-			(xy 193.04 33.02) (xy 200.66 33.02)
-		)
-		(stroke
-			(width 0)
-			(type default)
-		)
-	)
-	(wire
-		(pts
 			(xy 558.8 269.24) (xy 558.8 270.51)
 		)
@@
 	(wire
 		(pts
+			(xy 166.37 27.94) (xy 200.66 27.94)
+		)
+		(stroke
+			(width 0)
+			(type default)
+		)
+	)
+	(wire
+		(pts
 			(xy 252.73 392.43) (xy 252.73 397.51)
 		)
@@
 	(wire
 		(pts
-			(xy 193.04 25.4) (xy 200.66 25.4)
-		)
-		(stroke
-			(width 0)
-			(type default)
-		)
-	)
-	(wire
-		(pts
 			(xy 317.5 369.57) (xy 327.66 369.57)
 		)
@@
 	(wire
 		(pts
-			(xy 187.96 25.4) (xy 193.04 25.4)
-		)
-		(stroke
-			(width 0)
-			(type default)
-		)
-	)
-	(wire
-		(pts
 			(xy 314.96 214.63) (xy 303.53 214.63)
 		)
@@
 	(symbol
 		(lib_id "power:GND")
-		(at 200.66 38.1 0)
+		(at 200.66 34.29 0)
 		(unit 1)
 		(exclude_from_sim no)
@@
 		(dnp no)
 		(property "Reference" "#PWR047"
-			(at 200.66 44.45 0)
+			(at 200.66 40.64 0)
 			(effects
 				(font
@@
 		)
 		(property "Value" "GND"
-			(at 200.787 42.4942 0)
+			(at 200.787 38.6842 0)
 			(effects
 				(font
@@
 		)
 		(property "Footprint" ""
-			(at 200.66 38.1 0)
+			(at 200.66 34.29 0)
 			(effects
 				(font
@@
 		)
 		(property "Datasheet" ""
-			(at 200.66 38.1 0)
+			(at 200.66 34.29 0)
 			(effects
 				(font
@@
 		)
 		(property "Description" ""
-			(at 200.66 38.1 0)
+			(at 200.66 34.29 0)
 			(effects
 				(font
@@
 	(symbol
 		(lib_id "Connector:Conn_01x02_Socket")
-		(at 173.99 27.94 180)
+		(at 161.29 27.94 180)
 		(unit 1)
 		(exclude_from_sim no)
@@
 		(dnp no)
 		(property "Reference" "J10"
-			(at 174.498 22.606 0)
+			(at 161.798 22.606 0)
 			(effects
 				(font
@@
 		)
 		(property "Value" "Main_Supply"
-			(at 161.798 26.416 0)
+			(at 149.098 26.416 0)
 			(effects
 				(font
@@
 		)
 		(property "Footprint" ""
-			(at 173.99 27.94 0)
+			(at 161.29 27.94 0)
 			(effects
 				(font
@@
 		)
 		(property "Datasheet" "~"
-			(at 173.99 27.94 0)
+			(at 161.29 27.94 0)
 			(effects
 				(font
@@
 		)
 		(property "Description" "Generic connector, single row, 01x02, script generated"
-			(at 173.99 27.94 0)
+			(at 161.29 27.94 0)
 			(effects
 				(font
@@
 	(symbol
 		(lib_id "Diode:1N53xxB")
-		(at 193.04 29.21 270)
+		(at 191.77 25.4 180)
 		(unit 1)
 		(exclude_from_sim no)
@@
 		(fields_autoplaced yes)
 		(property "Reference" "D15"
-			(at 195.58 27.9399 90)
+			(at 191.77 19.05 0)
 			(effects
 				(font
 					(size 1.27 1.27)
 				)
-				(justify left)
 			)
 		)
 		(property "Value" "1N5242"
-			(at 195.58 30.4799 90)
+			(at 191.77 21.59 0)
 			(effects
 				(font
 					(size 1.27 1.27)
 				)
-				(justify left)
 			)
 		)
 		(property "Footprint" "Diode_THT:D_DO-201_P15.24mm_Horizontal"
-			(at 188.595 29.21 0)
+			(at 191.77 20.955 0)
 			(effects
 				(font
@@
 		)
 		(property "Datasheet" "https://diotec.com/tl_files/diotec/files/pdf/datasheets/1n5345b.pdf"
-			(at 193.04 29.21 0)
+			(at 191.77 25.4 0)
 			(effects
 				(font
@@
 		)
 		(property "Description" "5000mW Zener Diode, DO-201"
-			(at 193.04 29.21 0)
+			(at 191.77 25.4 0)
 			(effects
 				(font
@@
 	(symbol
 		(lib_id "Device:Fuse_Small")
-		(at 185.42 25.4 0)
+		(at 181.61 25.4 0)
 		(unit 1)
 		(exclude_from_sim no)
@@
 		(fields_autoplaced yes)
 		(property "Reference" "F1"
-			(at 185.42 20.32 0)
+			(at 181.61 20.32 0)
 			(effects
 				(font
@@
 		)
 		(property "Value" "Fuse"
-			(at 185.42 22.86 0)
+			(at 181.61 22.86 0)
 			(effects
 				(font
@@
 		)
 		(property "Footprint" ""
-			(at 185.42 25.4 0)
+			(at 181.61 25.4 0)
 			(effects
 				(font
@@
 		)
 		(property "Datasheet" "~"
-			(at 185.42 25.4 0)
+			(at 181.61 25.4 0)
 			(effects
 				(font
@@
 		)
 		(property "Description" "Fuse, small symbol"
-			(at 185.42 25.4 0)
+			(at 181.61 25.4 0)
 			(effects
 				(font
