File: Shield_VCU_Board/Shield_VCU_Board.kicad_sch (KiCad schematic)
At the start: 184 parts, among them J1 Conn_02x10_Odd_Even, J10 Main_Supply, J11 Molex_connector_40pin, J12 TFT Wire, J13 Molex_x06_Socket, J15 Conn_01x04_Socket, J2 Conn_02x10_Odd_Even, J3 Conn_02x09_Odd_Even, J4 Conn_02x09_Odd_Even, J5 Conn_02x09_Odd_Even, J6 Conn_02x10_Odd_Even, J7 Button_Activation_Logic, J8 Conn_ToSpeaker, J9 Wire_x06_Pin, U1 AS1115-BSST, U2 SN74LVC1G125DBV, U3 MC74HC14A, U4 TPA6205A1, U5 TLV76133DCY, U6 TLV76150DCY, U7 FT812, U8 TLV76133DCY, U9 TLV76133DCY, Y1 12MHz, Y2 SGM3766YTN5G

Commit message: Added proto footprints for Layout
Parts:
- removed TPH2: VCC+, symbol Connector:Conn_01x01_Socket
- added TPH2: VCC+, Connector_PinSocket_1.27mm:PinSocket_1x01_P1.27mm_Vertical, symbol Connector:Conn_01x01_Pin
- AUDIOL1, AUDV3.3, BKLTV5, CAN_H1, CAN_L1, CS1, DSPLV3.3, INT1, IRQ7, MISO1, MOSI1, PD1, SCK1, SCL7, SDA7, SEGV3.3, V12: footprint (none) -> TestPoint:TestPoint_Pad_D1.0mm
- C1, C10, C11, C12, C14, C15, C16, C17, C18, C19, C2, C20, C21, C22, C23, C24, C25, C26, C27, C28, C29, C3, C30, C31, C32, C33, C34, C35, C36, C37, C4, C40, C41, C42, C5, C6, C7, C9: footprint (none) -> Capacitor_SMD:C_0805_2012Metric_Pad1.18x1.45mm_HandSolder
- C13, C8: footprint (none) -> Capacitor_THT:CP_Radial_D5.0mm_P2.50mm
- D1, D2, D3, D4: footprint (none) -> LED_SMD:LED_1812_4532Metric_Pad1.30x3.40mm_HandSolder
- D11, D12, D13, D14: footprint (none) -> LED_SMD:LED_0805_2012Metric_Pad1.15x1.40mm_HandSolder
- F1: footprint (none) -> Fuse:Fuse_1206_3216Metric
- FB1, FB2: footprint (none) -> Inductor_SMD:L_Neosid_SM-PIC0512H
- H1, H2, H3, H4, H5, H6, H7, H8: footprint (none) -> MountingHole:MountingHole_2.7mm_M2.5_Pad
- J1, J2, J3, J4, J5, J6: footprint (none) -> Connector_PinHeader_1.00mm:PinHeader_2x18_P1.00mm_Vertical
- J10: footprint (none) -> Connector_Phoenix_GMSTB:PhoenixContact_GMSTBA_2,5_2-G-7,62_1x02_P7.62mm_Horizontal
- J11: footprint (none) -> Connector_FFC-FPC:Amphenol_F32Q-1A7x1-11040_1x40-1MP_P0.5mm_Horizontal
- J13: footprint (none) -> Connector_FFC-FPC:Molex_200528-0060_1x06-1MP_P1.00mm_Horizontal
- J15: footprint (none) -> Connector_Phoenix_GMSTB:PhoenixContact_GMSTBV_2,5_4-GF-7,62_1x04_P7.62mm_Vertical_ThreadedFlange
- J7: footprint (none) -> Connector_PinSocket_2.00mm:PinSocket_2x01_P2.00mm_Vertical_SMD
- J8: footprint (none) -> Connector_Phoenix_GMSTB:PhoenixContact_GMSTBVA_2,5_2-G-7,62_1x02_P7.62mm_Vertical
- L1: footprint (none) -> Inductor_SMD:L_TDK_VLF10040
- R1, R10, R11, R12, R13, R14, R15, R16, R17, R18, R2, R20, R21, R22, R23, R24, R25, R26, R27, R28, R29, R3, R30, R31, R32, R33, R34, R35, R36, R37, R38, R39, R4, R40, R41, R42, R43, R44, R45, R46, R47, R48, R49, R5, R50, R51, R52, R53, R54, R55, R56, R57, R58, R59, R6, R60, R61, R62, R63, R64, R7, R8, R9, RSET1: footprint (none) -> Resistor_SMD:R_1206_3216Metric_Pad1.30x1.75mm_HandSolder
- U4: footprint (none) -> Package_SON:SON-8-1EP_3x2mm_P0.5mm_EP1.4x1.6mm
- U7: footprint (none) -> Package_CSP:LFCSP-56-1EP_8x8mm_P0.5mm_EP6.6x6.6mm
- Y1: footprint (none) -> Crystal:Resonator-3Pin_W7.0mm_H2.5mm
Connections:
- net +12V: now also TPH2.1 (Pin_1)

Commit message: Layout proto_check
Parts:
- J1, J2, J3, J4, J5, J6: footprint Connector_PinHeader_1.00mm:PinHeader_2x18_P1.00mm_Vertical -> Connector_PinHeader_1.00mm:PinHeader_2x08_P1.00mm_Vertical
- R23, R24, R25, R26, R27, R28, R29, R30, R31, R32, R33, R34, R35, R36, R37, R38, R39, R40, R41, R42, R43, R44, R45, R46, R47, R48, R49, R50, R51: footprint Resistor_SMD:R_1206_3216Metric_Pad1.30x1.75mm_HandSolder -> Resistor_SMD:R_0201_0603Metric_Pad0.64x0.40mm_HandSolder
Changed lines of the file:
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@@
 			)
 		)
-		(property "Footprint" "Resistor_SMD:R_1206_3216Metric_Pad1.30x1.75mm_HandSolder"
+		(property "Footprint" "Resistor_SMD:R_0201_0603Metric_Pad0.64x0.40mm_HandSolder"
 			(at 481.33 120.65 0)
 			(effects
@@
 			)
 		)
-		(property "Footprint" "Resistor_SMD:R_1206_3216Metric_Pad1.30x1.75mm_HandSolder"
+		(property "Footprint" "Resistor_SMD:R_0201_0603Metric_Pad0.64x0.40mm_HandSolder"
 			(at 481.33 90.17 0)
 			(effects
@@
 			)
 		)
-		(property "Footprint" "Resistor_SMD:R_1206_3216Metric_Pad1.30x1.75mm_HandSolder"
+		(property "Footprint" "Resistor_SMD:R_0201_0603Metric_Pad0.64x0.40mm_HandSolder"
 			(at 481.33 95.25 0)
 			(effects
@@
 			)
 		)
-		(property "Footprint" "Resistor_SMD:R_1206_3216Metric_Pad1.30x1.75mm_HandSolder"
+		(property "Footprint" "Resistor_SMD:R_0201_0603Metric_Pad0.64x0.40mm_HandSolder"
 			(at 481.33 138.43 0)
 			(effects
@@
 			)
 		)
-		(property "Footprint" "Connector_PinHeader_1.00mm:PinHeader_2x18_P1.00mm_Vertical"
+		(property "Footprint" "Connector_PinHeader_1.00mm:PinHeader_2x08_P1.00mm_Vertical"
 			(at 121.92 113.03 0)
 			(effects
@@
 			)
 		)
-		(property "Footprint" "Resistor_SMD:R_1206_3216Metric_Pad1.30x1.75mm_HandSolder"
+		(property "Footprint" "Resistor_SMD:R_0201_0603Metric_Pad0.64x0.40mm_HandSolder"
 			(at 481.33 80.01 0)
 			(effects
@@
 			)
 		)
-		(property "Footprint" "Resistor_SMD:R_1206_3216Metric_Pad1.30x1.75mm_HandSolder"
+		(property "Footprint" "Resistor_SMD:R_0201_0603Metric_Pad0.64x0.40mm_HandSolder"
 			(at 481.33 105.41 0)
 			(effects
@@
 			)
 		)
-		(property "Footprint" "Resistor_SMD:R_1206_3216Metric_Pad1.30x1.75mm_HandSolder"
+		(property "Footprint" "Resistor_SMD:R_0201_0603Metric_Pad0.64x0.40mm_HandSolder"
 			(at 481.33 123.19 0)
 			(effects
@@
 			)
 		)
-		(property "Footprint" "Resistor_SMD:R_1206_3216Metric_Pad1.30x1.75mm_HandSolder"
+		(property "Footprint" "Resistor_SMD:R_0201_0603Metric_Pad0.64x0.40mm_HandSolder"
 			(at 481.33 107.95 0)
 			(effects
@@
 			)
 		)
-		(property "Footprint" "Resistor_SMD:R_1206_3216Metric_Pad1.30x1.75mm_HandSolder"
+		(property "Footprint" "Resistor_SMD:R_0201_0603Metric_Pad0.64x0.40mm_HandSolder"
 			(at 481.33 77.47 0)
 			(effects
@@
 			)
 		)
-		(property "Footprint" "Resistor_SMD:R_1206_3216Metric_Pad1.30x1.75mm_HandSolder"
+		(property "Footprint" "Resistor_SMD:R_0201_0603Metric_Pad0.64x0.40mm_HandSolder"
 			(at 481.33 143.51 0)
 			(effects
@@
 			)
 		)
-		(property "Footprint" "Resistor_SMD:R_1206_3216Metric_Pad1.30x1.75mm_HandSolder"
+		(property "Footprint" "Resistor_SMD:R_0201_0603Metric_Pad0.64x0.40mm_HandSolder"
 			(at 481.33 69.85 0)
 			(effects
@@
 			)
 		)
-		(property "Footprint" "Resistor_SMD:R_1206_3216Metric_Pad1.30x1.75mm_HandSolder"
+		(property "Footprint" "Resistor_SMD:R_0201_0603Metric_Pad0.64x0.40mm_HandSolder"
 			(at 481.33 87.63 0)
 			(effects
@@
 			)
 		)
-		(property "Footprint" "Resistor_SMD:R_1206_3216Metric_Pad1.30x1.75mm_HandSolder"
+		(property "Footprint" "Resistor_SMD:R_0201_0603Metric_Pad0.64x0.40mm_HandSolder"
 			(at 481.33 118.11 0)
 			(effects
@@
 			)
 		)
-		(property "Footprint" "Resistor_SMD:R_1206_3216Metric_Pad1.30x1.75mm_HandSolder"
+		(property "Footprint" "Resistor_SMD:R_0201_0603Metric_Pad0.64x0.40mm_HandSolder"
 			(at 481.33 125.73 0)
 			(effects
@@
 			)
 		)
-		(property "Footprint" "Resistor_SMD:R_1206_3216Metric_Pad1.30x1.75mm_HandSolder"
+		(property "Footprint" "Resistor_SMD:R_0201_0603Metric_Pad0.64x0.40mm_HandSolder"
 			(at 481.33 115.57 0)
 			(effects
@@
 			)
 		)
-		(property "Footprint" "Resistor_SMD:R_1206_3216Metric_Pad1.30x1.75mm_HandSolder"
+		(property "Footprint" "Resistor_SMD:R_0201_0603Metric_Pad0.64x0.40mm_HandSolder"
 			(at 481.33 72.39 0)
 			(effects
@@
 			)
 		)
-		(property "Footprint" "Resistor_SMD:R_1206_3216Metric_Pad1.30x1.75mm_HandSolder"
+		(property "Footprint" "Resistor_SMD:R_0201_0603Metric_Pad0.64x0.40mm_HandSolder"
 			(at 481.33 128.27 0)
 			(effects
@@
 			)
 		)
-		(property "Footprint" "Resistor_SMD:R_1206_3216Metric_Pad1.30x1.75mm_HandSolder"
+		(property "Footprint" "Resistor_SMD:R_0201_0603Metric_Pad0.64x0.40mm_HandSolder"
 			(at 481.33 140.97 0)
 			(effects
@@
 			)
 		)
-		(property "Footprint" "Resistor_SMD:R_1206_3216Metric_Pad1.30x1.75mm_HandSolder"
+		(property "Footprint" "Resistor_SMD:R_0201_0603Metric_Pad0.64x0.40mm_HandSolder"
 			(at 481.33 133.35 0)
 			(effects
@@
 			)
 		)
-		(property "Footprint" "Resistor_SMD:R_1206_3216Metric_Pad1.30x1.75mm_HandSolder"
+		(property "Footprint" "Resistor_SMD:R_0201_0603Metric_Pad0.64x0.40mm_HandSolder"
 			(at 481.33 113.03 0)
 			(effects
@@
 			)
 		)
-		(property "Footprint" "Connector_PinHeader_1.00mm:PinHeader_2x18_P1.00mm_Vertical"
+		(property "Footprint" "Connector_PinHeader_1.00mm:PinHeader_2x08_P1.00mm_Vertical"
 			(at 83.82 143.51 0)
 			(effects
@@
 			)
 		)
-		(property "Footprint" "Resistor_SMD:R_1206_3216Metric_Pad1.30x1.75mm_HandSolder"
+		(property "Footprint" "Resistor_SMD:R_0201_0603Metric_Pad0.64x0.40mm_HandSolder"
 			(at 481.33 74.93 0)
 			(effects
@@
 			)
 		)
-		(property "Footprint" "Resistor_SMD:R_1206_3216Metric_Pad1.30x1.75mm_HandSolder"
+		(property "Footprint" "Resistor_SMD:R_0201_0603Metric_Pad0.64x0.40mm_HandSolder"
 			(at 481.33 92.71 0)
 			(effects
@@
 			)
 		)
-		(property "Footprint" "Resistor_SMD:R_1206_3216Metric_Pad1.30x1.75mm_HandSolder"
+		(property "Footprint" "Resistor_SMD:R_0201_0603Metric_Pad0.64x0.40mm_HandSolder"
 			(at 481.33 102.87 0)
 			(effects
@@
 			)
 		)
-		(property "Footprint" "Connector_PinHeader_1.00mm:PinHeader_2x18_P1.00mm_Vertical"
+		(property "Footprint" "Connector_PinHeader_1.00mm:PinHeader_2x08_P1.00mm_Vertical"
 			(at 83.82 171.45 0)
 			(effects
@@
 			)
 		)
-		(property "Footprint" "Resistor_SMD:R_1206_3216Metric_Pad1.30x1.75mm_HandSolder"
+		(property "Footprint" "Resistor_SMD:R_0201_0603Metric_Pad0.64x0.40mm_HandSolder"
 			(at 481.33 82.55 0)
 			(effects
@@
 			)
 		)
-		(property "Footprint" "Connector_PinHeader_1.00mm:PinHeader_2x18_P1.00mm_Vertical"
+		(property "Footprint" "Connector_PinHeader_1.00mm:PinHeader_2x08_P1.00mm_Vertical"
 			(at 121.92 143.51 0)
 			(effects
@@
 			)
 		)
-		(property "Footprint" "Resistor_SMD:R_1206_3216Metric_Pad1.30x1.75mm_HandSolder"
+		(property "Footprint" "Resistor_SMD:R_0201_0603Metric_Pad0.64x0.40mm_HandSolder"
 			(at 481.33 110.49 0)
 			(effects
@@
 			)
 		)
-		(property "Footprint" "Resistor_SMD:R_1206_3216Metric_Pad1.30x1.75mm_HandSolder"
+		(property "Footprint" "Resistor_SMD:R_0201_0603Metric_Pad0.64x0.40mm_HandSolder"
 			(at 481.33 135.89 0)
 			(effects
@@
 			)
 		)
-		(property "Footprint" "Resistor_SMD:R_1206_3216Metric_Pad1.30x1.75mm_HandSolder"
+		(property "Footprint" "Resistor_SMD:R_0201_0603Metric_Pad0.64x0.40mm_HandSolder"
 			(at 481.33 100.33 0)
 			(effects
@@
 			)
 		)
-		(property "Footprint" "Connector_PinHeader_1.00mm:PinHeader_2x18_P1.00mm_Vertical"
+		(property "Footprint" "Connector_PinHeader_1.00mm:PinHeader_2x08_P1.00mm_Vertical"
 			(at 83.82 113.03 0)
 			(effects
@@
 			)
 		)
-		(property "Footprint" "Resistor_SMD:R_1206_3216Metric_Pad1.30x1.75mm_HandSolder"
+		(property "Footprint" "Resistor_SMD:R_0201_0603Metric_Pad0.64x0.40mm_HandSolder"
 			(at 481.33 97.79 0)
 			(effects
@@
 			)
 		)
-		(property "Footprint" "Resistor_SMD:R_1206_3216Metric_Pad1.30x1.75mm_HandSolder"
+		(property "Footprint" "Resistor_SMD:R_0201_0603Metric_Pad0.64x0.40mm_HandSolder"
 			(at 481.33 85.09 0)
 			(effects
@@
 			)
 		)
-		(property "Footprint" "Connector_PinHeader_1.00mm:PinHeader_2x18_P1.00mm_Vertical"
+		(property "Footprint" "Connector_PinHeader_1.00mm:PinHeader_2x08_P1.00mm_Vertical"
 			(at 121.92 172.72 0)
 			(effects

Commit message: New BL chip proto
New chip is currently placed but surrounding components not fine-selected
Parts:
- added C38: 4.7uF, Capacitor_SMD:C_0805_2012Metric_Pad1.18x1.45mm_HandSolder, symbol Device:C_Small
- added C39, C43: 1uF, Capacitor_SMD:C_0805_2012Metric_Pad1.18x1.45mm_HandSolder, symbol Device:C_Small
- added C44: 220nF, Capacitor_SMD:C_0805_2012Metric_Pad1.18x1.45mm_HandSolder, symbol Device:C_Small
- added D16: MBRS340, Diode_SMD:D_SMC, symbol Diode:MBRS340
- added D17: 1N4148WT, Diode_SMD:D_SOD-523, symbol Diode:1N4148WT
- added L2: 10uH, Inductor_SMD:L_TDK_VLF10040, symbol Device:L_Small
- added R19: 1k, Resistor_SMD:R_1206_3216Metric_Pad1.30x1.75mm_HandSolder, symbol Device:R_Small
- added R65: 0.57R, Resistor_SMD:R_1206_3216Metric_Pad1.30x1.75mm_HandSolder, symbol Device:R_Small
- added U10: TPS61165DBV, Package_TO_SOT_SMD:SOT-23-6, symbol Driver_LED:TPS61165DBV
Connections:
- net 5V_BKLT: now also C38.1, L2.1, R19.2
- net BL_PWM: now also U10.2 (CTRL)
- net GND: now also C38.2, C39.2, C43.2, C44.2, D17.2 (A), R65.1, U10.4 (GND)
- net LED_A: now also C43.1, D16.1 (K)
- net LED_K: now also R65.2, U10.6 (FB)
- new net: D16.2 (A), L2.2, U10.3 (SW)
- new net: C44.1, U10.5 (COMP)
- new net: C39.1, D17.1 (K), R19.1, U10.1 (VIN)
Other:
- note added: "NOT APPLICABLE !!! NO CHIP AVAILABLE"
- moved on the sheet: C21, C22, C23, C24, C25, C26, D5, D6, L1, R1, R17, R18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

Commit message: BL drive correction
Parts:
- removed C21: 10uF, Capacitor_SMD:C_0805_2012Metric_Pad1.18x1.45mm_HandSolder, symbol Device:C_Small
- removed C22, C26: 27pF, Capacitor_SMD:C_0805_2012Metric_Pad1.18x1.45mm_HandSolder, symbol Device:C_Small
- removed C23, C24: 1uF, Capacitor_SMD:C_0805_2012Metric_Pad1.18x1.45mm_HandSolder, symbol Device:C_Small
- removed C25: 0.1uF, Capacitor_SMD:C_0805_2012Metric_Pad1.18x1.45mm_HandSolder, symbol Device:C_Small
- removed D5: MBR0540, Diode_SMD:D_SOD-123, symbol Diode:MBR0540
- removed D6: 3SMAJ5935B-TP, Diode_SMD:D_SOD-123, symbol Diode:MBR0540
- removed L1: 10uH, Inductor_SMD:L_TDK_VLF10040, symbol Device:L_Small
- removed R1: 47k, Resistor_SMD:R_1206_3216Metric_Pad1.30x1.75mm_HandSolder, symbol Device:R_Small
- removed R17: 1.69 1%, Resistor_SMD:R_1206_3216Metric_Pad1.30x1.75mm_HandSolder, symbol Device:R_Small
- removed R18: 3.3 1%, Resistor_SMD:R_1206_3216Metric_Pad1.30x1.75mm_HandSolder, symbol Device:R_Small
- removed Y2: SGM3766YTN5G, Oscillator:Oscillator_SMD_SeikoEpson_SG8002CE-4Pin_3.2x2.5mm, symbol A_GHST_Lib:SGM3766YTN5G
- RSET: renamed from R65; value 0.57R -> 1.1R1%
Other:
- note removed: "NOT APPLICABLE !!! NO CHIP AVAILABLE"

Commit message: PCL_Layout_Arrangements
Initial PCB components arangement done.
Not a functional version!
Parts:
- added RN_Sample_1: R_Pack04, symbol Device:R_Pack04
- J15: footprint Connector_Phoenix_GMSTB:PhoenixContact_GMSTBV_2,5_4-GF-7,62_1x04_P7.62mm_Vertical_ThreadedFlange -> Connector_PinHeader_1.00mm:PinHeader_1x04_P1.00mm_Vertical
- renumbered RSET to RSET2
Connections:
- net 3V3_AUD: now also R53.1
- net 3V3_SPKR: no longer R53.1
Other:
- moved on the sheet: D17
Changed lines of the file:
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@@
 	(wire
 		(pts
-			(xy 280.67 401.32) (xy 280.67 382.27)
+			(xy 280.67 402.59) (xy 280.67 382.27)
 		)
 		(stroke
@@
 	(wire
 		(pts
+			(xy 273.05 389.89) (xy 273.05 391.16)
+		)
+		(stroke
+			(width 0)
+			(type default)
+		)
+	)
+	(wire
+		(pts
 			(xy 469.9 80.01) (xy 469.9 85.09)
 		)
@@
 	(wire
 		(pts
-			(xy 273.05 383.54) (xy 273.05 379.73)
+			(xy 273.05 382.27) (xy 273.05 379.73)
 		)
 		(stroke
@@
 	(wire
 		(pts
-			(xy 262.89 401.32) (xy 280.67 401.32)
+			(xy 262.89 402.59) (xy 280.67 402.59)
 		)
 		(stroke
@@
 	(global_label "BL_PWM"
 		(shape input)
-		(at 262.89 401.32 180)
+		(at 262.89 402.59 180)
 		(effects
 			(font
@@
 		)
 		(property "Intersheetrefs" "${INTERSHEET_REFS}"
-			(at 262.89 401.32 0)
+			(at 262.89 402.59 0)
 			(effects
 				(font
@@
 		(on_board yes)
 		(dnp no)
-		(property "Reference" "RSET"
+		(property "Reference" "RSET2"
 			(at 322.072 391.668 0)
 			(effects
@@
 			(project "Shield_VCU_Board"
 				(path "/4a8cb20d-5f30-4163-a2c8-18e2deeb65d3"
-					(reference "RSET")
+					(reference "RSET2")
 					(unit 1)
 				)
@@
 		(dnp no)
 		(property "Reference" "J10"
-			(at 22.098 238.506 0)
+			(at 18.034 242.316 0)
 			(effects
 				(font
@@
 		)
 		(property "Value" "Main_Supply"
-			(at 18.542 246.38 90)
+			(at 21.082 238.506 0)
 			(effects
 				(font
@@
 	)
 	(symbol
+		(lib_id "Device:R_Pack04")
+		(at 92.71 345.44 90)
+		(unit 1)
+		(exclude_from_sim no)
+		(in_bom yes)
+		(on_board yes)
+		(dnp no)
+		(fields_autoplaced yes)
+		(property "Reference" "RN_Sample_1"
+			(at 92.71 336.55 90)
+			(effects
+				(font
+					(size 1.27 1.27)
+				)
+			)
+		)
+		(property "Value" "R_Pack04"
+			(at 92.71 339.09 90)
+			(effects
+				(font
+					(size 1.27 1.27)
+				)
+			)
+		)
+		(property "Footprint" ""
+			(at 92.71 338.455 90)
+			(effects
+				(font
+					(size 1.27 1.27)
+				)
+				(hide yes)
+			)
+		)
+		(property "Datasheet" "~"
+			(at 92.71 345.44 0)
+			(effects
+				(font
+					(size 1.27 1.27)
+				)
+				(hide yes)
+			)
+		)
+		(property "Description" "4 resistor network, parallel topology"
+			(at 92.71 345.44 0)
+			(effects
+				(font
+					(size 1.27 1.27)
+				)
+				(hide yes)
+			)
+		)
+		(pin "5"
+		)
+		(pin "3"
+		)
+		(pin "6"
+		)
+		(pin "8"
+		)
+		(pin "1"
+		)
+		(pin "7"
+		)
+		(pin "2"
+		)
+		(pin "4"
+		)
+		(instances
+			(project ""
+				(path "/4a8cb20d-5f30-4163-a2c8-18e2deeb65d3"
+					(reference "RN_Sample_1")
+					(unit 1)
+				)
+			)
+		)
+	)
+	(symbol
 		(lib_id "power:GND")
 		(at 393.7 198.12 0)
@@
 	(symbol
 		(lib_id "Diode:1N4148WT")
-		(at 273.05 387.35 270)
+		(at 273.05 386.08 270)
 		(unit 1)
 		(exclude_from_sim no)
@@
 		(dnp no)
 		(property "Reference" "D17"
-			(at 269.24 384.81 90)
+			(at 269.24 383.54 90)
 			(effects
 				(font
@@
 		)
 		(property "Value" "1N4148WT"
-			(at 275.844 381.508 0)
+			(at 275.59 381.508 0)
 			(effects
 				(font
@@
 		)
 		(property "Footprint" "Diode_SMD:D_SOD-523"
-			(at 268.605 387.35 0)
+			(at 268.605 386.08 0)
 			(effects
 				(font
@@
 		)
 		(property "Datasheet" "https://www.diodes.com/assets/Datasheets/ds30396.pdf"
-			(at 273.05 387.35 0)
+			(at 273.05 386.08 0)
 			(effects
 				(font
@@
 		)
 		(property "Description" "75V 0.15A Fast switching Diode, SOD-523"
-			(at 273.05 387.35 0)
+			(at 273.05 386.08 0)
 			(effects
 				(font
@@
 		)
 		(property "Sim.Device" "D"
-			(at 273.05 387.35 0)
+			(at 273.05 386.08 0)
 			(effects
 				(font
@@
 		)
 		(property "Sim.Pins" "1=K 2=A"
-			(at 273.05 387.35 0)
+			(at 273.05 386.08 0)
 			(effects
 				(font
@@
 			)
 		)
-		(property "Footprint" "Connector_Phoenix_GMSTB:PhoenixContact_GMSTBV_2,5_4-GF-7,62_1x04_P7.62mm_Vertical_ThreadedFlange"
+		(property "Footprint" "Connector_PinHeader_1.00mm:PinHeader_1x04_P1.00mm_Vertical"
 			(at 113.03 85.09 0)
 			(effects
@@
 			)
 		)
-		(property "Value" "3V3_SPKR"
+		(property "Value" "3V3_AUD"
 			(at 60.071 278.8158 0)
 			(effects

Commit message: Layout_Progress_0.1
Parts:
- J1, J2, J3, J4, J5, J6: footprint Connector_PinHeader_1.00mm:PinHeader_2x08_P1.00mm_Vertical -> Connector_PinHeader_2.54mm:PinHeader_2x10_P2.54mm_Vertical
Changed lines of the file:
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@@
 			)
 		)
-		(property "Footprint" "Connector_PinHeader_1.00mm:PinHeader_2x08_P1.00mm_Vertical"
+		(property "Footprint" "Connector_PinHeader_2.54mm:PinHeader_2x10_P2.54mm_Vertical"
 			(at 121.92 113.03 0)
 			(effects
@@
 			)
 		)
-		(property "Footprint" "Connector_PinHeader_1.00mm:PinHeader_2x08_P1.00mm_Vertical"
+		(property "Footprint" "Connector_PinHeader_2.54mm:PinHeader_2x10_P2.54mm_Vertical"
 			(at 83.82 143.51 0)
 			(effects
@@
 			)
 		)
-		(property "Footprint" "Connector_PinHeader_1.00mm:PinHeader_2x08_P1.00mm_Vertical"
+		(property "Footprint" "Connector_PinHeader_2.54mm:PinHeader_2x10_P2.54mm_Vertical"
 			(at 83.82 171.45 0)
 			(effects
@@
 			)
 		)
-		(property "Footprint" "Connector_PinHeader_1.00mm:PinHeader_2x08_P1.00mm_Vertical"
+		(property "Footprint" "Connector_PinHeader_2.54mm:PinHeader_2x10_P2.54mm_Vertical"
 			(at 121.92 143.51 0)
 			(effects
@@
 			)
 		)
-		(property "Footprint" "Connector_PinHeader_1.00mm:PinHeader_2x08_P1.00mm_Vertical"
+		(property "Footprint" "Connector_PinHeader_2.54mm:PinHeader_2x10_P2.54mm_Vertical"
 			(at 83.82 113.03 0)
 			(effects
@@
 			)
 		)
-		(property "Footprint" "Connector_PinHeader_1.00mm:PinHeader_2x08_P1.00mm_Vertical"
+		(property "Footprint" "Connector_PinHeader_2.54mm:PinHeader_2x10_P2.54mm_Vertical"
 			(at 121.92 172.72 0)
 			(effects

Commit message: Layout_Progress_0.2
+ 7seg x8 Digits connected
+LDO started
Parts:
- L2: footprint Inductor_SMD:L_TDK_VLF10040 -> Inductor_SMD:L_TDK_SLF7032
Changed lines of the file:
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@@
 			)
 		)
-		(property "Footprint" "Inductor_SMD:L_TDK_VLF10040"
+		(property "Footprint" "Inductor_SMD:L_TDK_SLF7032"
 			(at 298.45 370.84 0)
 			(effects

Commit message: Layout_progress_0.3
Parts:
- 7U1, 7U2, 7U3, 7U4, 7U5, 7U6, 7U7, 7U8: footprint Display_7Segment:HDSP-7801 -> GHSTProj:T7DS052BC
- J10: footprint Connector_Phoenix_GMSTB:PhoenixContact_GMSTBA_2,5_2-G-7,62_1x02_P7.62mm_Horizontal -> Connector_Molex:Molex_KK-396_A-41792-0002_1x02_P3.96mm_Horizontal
- J8: footprint Connector_Phoenix_GMSTB:PhoenixContact_GMSTBVA_2,5_2-G-7,62_1x02_P7.62mm_Vertical -> Connector_PinSocket_2.54mm:PinSocket_1x02_P2.54mm_Horizontal
- J9, RTP1: now left out of the parts list
Changed lines of the file:
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@@
 			)
 		)
-		(property "Footprint" "Display_7Segment:HDSP-7801"
+		(property "Footprint" "GHSTProj:T7DS052BC"
 			(at 322.58 114.3 0)
 			(effects
@@
 			)
 		)
-		(property "Footprint" "Display_7Segment:HDSP-7801"
+		(property "Footprint" "GHSTProj:T7DS052BC"
 			(at 322.58 260.35 0)
 			(effects
@@
 			)
 		)
-		(property "Footprint" "Display_7Segment:HDSP-7801"
+		(property "Footprint" "GHSTProj:T7DS052BC"
 			(at 322.58 231.14 0)
 			(effects
@@
 		(unit 1)
 		(exclude_from_sim no)
-		(in_bom yes)
-		(on_board yes)
+		(in_bom no)
+		(on_board no)
 		(dnp no)
 		(property "Reference" "RTP1"
@@
 			)
 		)
-		(property "Footprint" "Display_7Segment:HDSP-7801"
+		(property "Footprint" "GHSTProj:T7DS052BC"
 			(at 322.58 55.88 0)
 			(effects
@@
 			)
 		)
-		(property "Footprint" "Display_7Segment:HDSP-7801"
+		(property "Footprint" "GHSTProj:T7DS052BC"
 			(at 322.58 143.51 0)
 			(effects
@@
 			)
 		)
-		(property "Footprint" "Connector_Phoenix_GMSTB:PhoenixContact_GMSTBA_2,5_2-G-7,62_1x02_P7.62mm_Horizontal"
+		(property "Footprint" "Connector_Molex:Molex_KK-396_A-41792-0002_1x02_P3.96mm_Horizontal"
 			(at 21.59 243.84 0)
 			(effects
@@
 			)
 		)
-		(property "Footprint" "Connector_Phoenix_GMSTB:PhoenixContact_GMSTBVA_2,5_2-G-7,62_1x02_P7.62mm_Vertical"
+		(property "Footprint" "Connector_PinSocket_2.54mm:PinSocket_1x02_P2.54mm_Horizontal"
 			(at 547.37 325.12 0)
 			(effects
@@
 			)
 		)
-		(property "Footprint" "Display_7Segment:HDSP-7801"
+		(property "Footprint" "GHSTProj:T7DS052BC"
 			(at 322.58 172.72 0)
 			(effects
@@
 			)
 		)
-		(property "Footprint" "Display_7Segment:HDSP-7801"
+		(property "Footprint" "GHSTProj:T7DS052BC"
 			(at 322.58 85.09 0)
 			(effects
@@
 			)
 		)
-		(property "Footprint" "Display_7Segment:HDSP-7801"
+		(property "Footprint" "GHSTProj:T7DS052BC"
 			(at 322.58 201.93 0)
 			(effects
@@
 		(unit 1)
 		(exclude_from_sim no)
-		(in_bom yes)
-		(on_board yes)
+		(in_bom no)
+		(on_board no)
 		(dnp no)
 		(property "Reference" "J9"
