File: Shield_VCU_Board/1.KiCad/Shield_VCU_Board.kicad_sch (KiCad schematic)
At the start: 187 parts, among them J1 Conn_02x08_Odd_Even, J10 Main_Supply, J11 Conn_01x40_Socket, J12 TFT Wire, J13 Conn_Molex_TouchPanel, J14 CAN_OUT, J15 Conn_01x04_Socket, J16 CAN_IN, J2 Conn_02x10_Odd_Even, J3/1 NXP3, J4 Conn_02x08_Odd_Even, J5 Conn_02x10_Odd_Even, J6 Conn_02x10_Odd_Even, J7 Button_Activation_Logic, J8 Conn_ToSpeaker, J9 Wire_x06_Pin, Q1 BSS138, Q2 BSS138, Q3 BSS138, Q4 BSS138, U1 AS1115-BSST, U10 TPS61165-Q1, U12 TPS54202DDC, U13 TPS54202DDC, U2 SN74LVC1G125DBV, U3 MC74HC14A, U4 TPA6211A1 - ?, U5 TLV76150DCY, U6 TLV76150DCY, U7 FT813Q, U8 TLV76133DCY, U9 TLV76133DCY

Commit message: Reworked segments routing
Parts:
- removed NT1: GNDTie, NetTie:NetTie-2_SMD_Pad2.0mm, symbol Device:NetTie_2
- removed R31, R32, R33, R34: 0R, Resistor_SMD:R_1206_3216Metric_Pad1.30x1.75mm_HandSolder, symbol Device:R_Small
- added JP1, JP2, JP3, JP4: SolderJumper_2_Bridged, Jumper:SolderJumper-2_P1.3mm_Open_TrianglePad1.0x1.5mm, symbol Jumper:SolderJumper_2_Bridged
Connections:
- net +3.7V: now also JP1.2 (B)
- net +5.3V: now also JP2.2 (B)
- net BAT+: now also JP3.1 (A), JP4.1 (A)
- net at C48.1, C52.1, L3.2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: now also JP1.1 (A)
- net at C47.1, C54.1, U12.3 (VIN): now also JP3.2 (B)
- net at C49.1, C55.1, U13.3 (VIN): now also JP4.2 (B)
- net at C51.1, C53.1, L4.2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: now also JP2.1 (A)

Commit message: Revamped connections and ground planes for the rest of the PCB
Parts:
- removed R29, R30: 0R, Resistor_SMD:R_1206_3216Metric_Pad1.30x1.75mm_HandSolder, symbol Device:R_Small
- added JP5, JP6: SolderJumper_2_Open, Jumper:SolderJumper-2_P1.3mm_Open_TrianglePad1.0x1.5mm, symbol Jumper:SolderJumper_2_Open
Connections:
- net +3.7V: now also JP6.2 (B); no longer C33.1, D10.1 (K), U9.3 (VI)
- net +5.3V: now also C33.1, D10.1 (K), U9.3 (VI), JP5.2 (B)
- net BAT+: now also JP5.1 (A), JP6.1 (A)
