File: Shield_VCU_Board/1.KiCad/Shield_VCU_Board.kicad_sch (KiCad schematic)
At the start: 186 parts, among them J1 Conn_02x08_Odd_Even, J10 Main_Supply, J11 Conn_01x40_Socket, J12 TFT Wire, J13 Conn_Molex_TouchPanel, J14 CAN_OUT, J15 Conn_01x04_Socket, J16 CAN_IN, J2 Conn_02x10_Odd_Even, J3/1 NXP3, J4 Conn_02x08_Odd_Even, J5 Conn_02x10_Odd_Even, J6 Conn_02x10_Odd_Even, J7 Button_Activation_Logic, J8 Conn_ToSpeaker, J9 Wire_x06_Pin, Q1 BSS138, Q2 BSS138, Q3 BSS138, Q4 BSS138, U1 AS1115-BSST, U10 TPS61165-Q1, U12 TPS54202DDC, U13 TPS54202DDC, U2 SN74LVC1G125DBV, U3 MC74HC14A, U4 TPA6211A1 - ?, U5 TLV76150DCY, U6 TLV76150DCY, U7 FT813Q, U8 TLV76133DCY, U9 TLV76133DCY

Commit message: BOM v2.0 - added
Parts:
- C48, C51, C52, C53: footprint Capacitor_SMD:C_0805_2012Metric_Pad1.18x1.45mm_HandSolder -> Capacitor_SMD:C_1210_3225Metric_Pad1.33x2.70mm_HandSolder
- L3, L4: footprint Inductor_SMD:L_Pulse_PA4340 -> Inductor_SMD:L_Coilcraft_LPS4018
- R2: value 634 -> 635R
Changed lines of the file:
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@@
 			)
 		)
-		(property "Footprint" "Capacitor_SMD:C_0805_2012Metric_Pad1.18x1.45mm_HandSolder"
+		(property "Footprint" "Capacitor_SMD:C_1210_3225Metric_Pad1.33x2.70mm_HandSolder"
 			(at 102.87 255.27 0)
 			(hide yes)
@@
 			)
 		)
-		(property "Footprint" "Inductor_SMD:L_Pulse_PA4340"
+		(property "Footprint" "Inductor_SMD:L_Coilcraft_LPS4018"
 			(at 90.17 250.19 0)
 			(hide yes)
@@
 			)
 		)
-		(property "Footprint" "Capacitor_SMD:C_0805_2012Metric_Pad1.18x1.45mm_HandSolder"
+		(property "Footprint" "Capacitor_SMD:C_1210_3225Metric_Pad1.33x2.70mm_HandSolder"
 			(at 104.14 303.53 0)
 			(hide yes)
@@
 			)
 		)
-		(property "Footprint" "Capacitor_SMD:C_0805_2012Metric_Pad1.18x1.45mm_HandSolder"
+		(property "Footprint" "Capacitor_SMD:C_1210_3225Metric_Pad1.33x2.70mm_HandSolder"
 			(at 109.22 255.27 0)
 			(hide yes)
@@
 			)
 		)
-		(property "Footprint" "Capacitor_SMD:C_0805_2012Metric_Pad1.18x1.45mm_HandSolder"
+		(property "Footprint" "Capacitor_SMD:C_1210_3225Metric_Pad1.33x2.70mm_HandSolder"
 			(at 111.76 303.53 0)
 			(hide yes)
@@
 			)
 		)
-		(property "Value" "634"
+		(property "Value" "635R"
 			(at 29.21 105.918 90)
 			(show_name no)
@@
 			)
 		)
-		(property "Footprint" "Inductor_SMD:L_Pulse_PA4340"
+		(property "Footprint" "Inductor_SMD:L_Coilcraft_LPS4018"
 			(at 92.71 295.91 0)
 			(hide yes)

Commit message: V2.21
Layout 1 ready
Parts:
- removed 3V7: 3V7, TestPoint:TestPoint_Pad_D1.0mm, symbol Connector:TestPoint
- removed AUDV5, BKLTV5: TestPoint, TestPoint:TestPoint_Pad_D1.0mm, symbol Connector:TestPoint
- removed C27, C29: 1uF, Capacitor_SMD:C_0805_2012Metric_Pad1.18x1.45mm_HandSolder, symbol Device:C_Small
- removed C28, C30: 2.2uF, Capacitor_SMD:C_0805_2012Metric_Pad1.18x1.45mm_HandSolder, symbol Device:C_Small
- removed C45, C54: 0.1uF, Capacitor_SMD:C_0805_2012Metric_Pad1.18x1.45mm_HandSolder, symbol Device:C_Small
- removed C47: 10uF, Capacitor_SMD:C_1210_3225Metric_Pad1.33x2.70mm_HandSolder, symbol Device:C_Small
- removed C48, C52: 22uF, Capacitor_SMD:C_1210_3225Metric_Pad1.33x2.70mm_HandSolder, symbol Device:C_Small
- removed D13, D14: LED, LED_SMD:LED_0805_2012Metric, symbol Device:LED
- removed D7, D8: MBR0540, Diode_SMD:D_SOD-123, symbol Diode:MBR0540
- removed L3: 10uH, Inductor_SMD:L_Coilcraft_LPS4018, symbol Device:L_Small
- removed NT1: GNDTie, NetTie:NetTie-2_SMD_Pad2.0mm, symbol Device:NetTie_2
- removed R30, R31, R33: 0R, Resistor_SMD:R_1206_3216Metric_Pad1.30x1.75mm_HandSolder, symbol Device:R_Small
- removed R53, R54: 1k, Resistor_SMD:R_1206_3216Metric_Pad1.30x1.75mm_HandSolder, symbol Device:R_Small
- removed R59: 523k, Resistor_SMD:R_1206_3216Metric_Pad1.30x1.75mm_HandSolder, symbol Device:R_Small
- removed R60: 100k, Resistor_SMD:R_1206_3216Metric_Pad1.30x1.75mm_HandSolder, symbol Device:R_Small
- removed U12: TPS54202DDC, Package_TO_SOT_SMD:SOT-23-6, symbol Regulator_Switching:TPS54202DDC
- removed U5: TLV76150DCY, Package_TO_SOT_SMD:SOT-223-3_TabPin2, symbol Regulator_Linear:TLV76133DCY
- removed U6: TLV76150DCY, Package_TO_SOT_SMD:SOT-223-3_TabPin2, symbol Regulator_Linear:TLV76150DCY
- added C15: 22uF, Capacitor_SMD:CP_Elec_5x5.4, symbol Device:C_Polarized
- added C21: 100uF, Capacitor_SMD:CP_Elec_5x5.4, symbol Device:C_Polarized
- R65: value 787k -> 73.2k
- R66: value 100k -> 10k
Connections:
- net +3.7V is gone; now on net +5.3V: C31.1, C33.1, D10.1 (K), D9.1 (K), U8.3 (VI), U9.3 (VI)
- net 5V_AUD is gone; now on net +5.3V: FB2.1
- net 5V_BKLT is gone; now on net +5.3V: C38.1, L2.1, R19.2
- net GND: now also C15.2, C21.2
- net at C49.1, C55.1, R32.1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: now also C15.1
- net at C51.1, C53.1, L4.2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: now also C21.1
- no-connect marks 121 -> 120
Other:
- note added: "LDO 3V3"
- note removed: "10V X7R ceramic"
- note removed: "BAT+ -> 3.7V"
- note removed: "LDO 3V3 & 5V"
- moved on the sheet: C31, C32, C33, C34, C49, C50, C51, C53, C55, D10, D11, D12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

Commit message: AUDIO chip footprint correction
Parts:
- U4: footprint TPA:TPS73601DRBR -> AUD:SOP65P490X110-9L
Changed lines of the file:
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@@
 			)
 		)
-		(property "Footprint" "TPA:TPS73601DRBR"
+		(property "Footprint" "AUD:SOP65P490X110-9L"
 			(at 513.08 347.98 0)
 			(hide yes)

Commit message: Routing optimisations
Parts:
- added C45: 0.1uF, Capacitor_SMD:C_0805_2012Metric_Pad1.18x1.45mm_HandSolder, symbol Device:C_Small
- added C46: 27pF, Capacitor_SMD:C_0805_2012Metric_Pad1.18x1.45mm_HandSolder, symbol Device:C_Small
Connections:
- net 3V3_DSPL: now also C45.1, C46.1
- net GND: now also C45.2, C46.2
- net at J13.3 (Pin_3), RN8.3 (R3.1): no longer R61.1
- net at J13.4 (Pin_4), RN8.4 (R4.1): no longer R63.1
- net at RN8.8 (R1.2), U7.23 (CTP_RST_N): now also R62.2
- net at RN8.7 (R2.2), U7.24 (CTP_INT_N): now also R64.1
- net at RN8.6 (R3.2), U7.25 (CTP_SCL): now also R63.1
- net at RN8.5 (R4.2), U7.26 (CTP_SDA): now also R61.1
- new net: J13.5 (Pin_5), RN8.1 (R1.1)
- new net: J13.6 (Pin_6), RN8.2 (R2.1)
Other:
- moved on the sheet: C16, C41, R61, R62, R63, R64, RN8

Commit message: Jumper added+ GND Sharp edges removed
Parts:
- removed R29, R32, R34: 0R, Resistor_SMD:R_1206_3216Metric_Pad1.30x1.75mm_HandSolder, symbol Device:R_Small
- added JP1, JP2: SolderJumper_2_Open, Jumper:SolderJumper-2_P1.3mm_Open_RoundedPad1.0x1.5mm, symbol Jumper:SolderJumper_2_Open
- added JP3: SolderJumper_2_Open, Jumper:SolderJumper-2_P1.3mm_Open_TrianglePad1.0x1.5mm, symbol Jumper:SolderJumper_2_Open
Connections:
- net +5.3V: now also JP1.2 (B), JP3.2 (B)
- net BAT+: now also JP2.1 (A), JP3.1 (A)
- net at C15.1, C49.1, C55.1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: now also JP2.2 (B)
- net at C21.1, C51.1, C53.1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: now also JP1.1 (A)
Other:
- note added: "Solder JP3, remove JP1 & JP2"
- note removed: "Remove R31,R32,R33,R34"
- moved on the sheet: C15, C21, C49, C50, C51, C53, C55, L4, R65, R66, U13
